File: Fuses.kicad_sch (KiCad schematic)
At the start: 24 parts, among them J2 Conn_01x02_Female, J3 Conn_01x02_Female, J4 Conn_01x02_Female, J5 Conn_01x02_Female, J6 Conn_01x02_Female, J7 Conn_01x02_Female, J8 Conn_01x02_Female, J9 Conn_01x02_Female

Commit message: Updated according to requirements
Parts:
- J2, J3, J4, J5, J6, J7, J8, J9: footprint Connector_JST:JST_XH_B2B-XH-AM_1x02_P2.50mm_Vertical -> Connector_JST:JST_XH_B2B-XH-A_1x02_P2.50mm_Vertical
Connections:
- net DRIVE_MOTORS_LEFT is gone; now on net GND: J2.2 (Pin_2), J5.2 (Pin_2), J6.2 (Pin_2)
- net DRIVE_MOTORS_RIGHT is gone; now on net GND: J3.2 (Pin_2), J7.2 (Pin_2), J9.2 (Pin_2)
- net AUX1_MOTORS1: no longer names the net of F3.2, F7.2, J4.1 (Pin_1)
- net AUX1_MOTORS2: no longer names the net of F4.2, F8.2, J5.1 (Pin_1)
- net AUX2_MOTORS1: no longer names the net of F11.2, F15.2, J8.1 (Pin_1)
- net AUX2_MOTORS2: no longer names the net of F12.2, F16.2, J9.1 (Pin_1)
- net AUX_MOTORS renamed GND
- net DRIVE_MOTOR_LEFT_FRONT: no longer names the net of F1.2, F5.2, J2.1 (Pin_1)
- net DRIVE_MOTOR_LEFT_REAR: no longer names the net of F13.2, F9.2, J6.1 (Pin_1)
- net DRIVE_MOTOR_RIGHT_FRONT: no longer names the net of F2.2, F6.2, J3.1 (Pin_1)
- net DRIVE_MOTOR_RIGHT_REAR: no longer names the net of F10.2, F14.2, J7.1 (Pin_1)

Commit message: Added 9V buck converter
Parts:
- added D1, D2, D3, D4, D5, D6, D7, D8: LED_Small, LED_SMD:LED_0603_1608Metric, symbol Device:LED_Small
- added R10, R3, R4, R5, R6, R7, R8, R9: 10k, Resistor_SMD:R_0603_1608Metric, symbol Device:R_US
- J2, J3, J4, J5, J6, J7, J8, J9: footprint Connector_JST:JST_XH_B2B-XH-A_1x02_P2.50mm_Vertical -> AndersonPowerPole:PowerPole_45A_Vert
Connections:
- net +24V: now also D1.2 (A), D2.2 (A), D3.2 (A), D4.2 (A), D5.2 (A), D6.2 (A), D7.2 (A), D8.2 (A)
- net DRIVE_MOTOR_LEFT_FRONT: now reaches F1.2, F5.2, J2.1 (Pin_1)
- net DRIVE_MOTOR_LEFT_FRONT: now also R3.2
- net PLUNGE_MOTOR: now reaches F12.2, F16.2, J9.1 (Pin_1)
- net PLUNGE_MOTOR: now also R10.2
- net GATE_LIFT_MOTOR_2: now reaches F11.2, F15.2, J8.1 (Pin_1)
- net GATE_LIFT_MOTOR_2: now also R9.2
- net DRIVE_MOTOR_RIGHT_REAR: now reaches F10.2, F14.2, J7.1 (Pin_1)
- net DRIVE_MOTOR_RIGHT_REAR: now also R8.2
- net GATE_LIFT_MOTOR_1: now reaches F3.2, F7.2, J4.1 (Pin_1)
- net GATE_LIFT_MOTOR_1: now also R5.2
- net DRIVE_MOTOR_RIGHT_FRONT: now reaches F2.2, F6.2, J3.1 (Pin_1)
- net DRIVE_MOTOR_RIGHT_FRONT: now also R4.2
- net DRIVE_MOTOR_LEFT_REAR: now reaches F13.2, F9.2, J6.1 (Pin_1)
- net DRIVE_MOTOR_LEFT_REAR: now also R7.2
- net DIG_MOTOR: now reaches F4.2, F8.2, J5.1 (Pin_1)
- net DIG_MOTOR: now also R6.2
- new net: D7.1 (K), R9.1
- new net: D2.1 (K), R4.1
- new net: D1.1 (K), R3.1
- new net: D6.1 (K), R8.1
- new net: D8.1 (K), R10.1
- new net: D4.1 (K), R6.1
- new net: D3.1 (K), R5.1
- new net: D5.1 (K), R7.1
Other:
- moved on the sheet: J2

Commit message: No point using Fuses w/o fuse holders, Also added 3D models
Parts:
- F1, F10, F11, F12, F13, F14, F15, F16, F2, F3, F4, F5, F6, F7, F8, F9: footprint Fuse:Fuse_Blade_Mini_directSolder -> Fuse:Fuseholder_Blade_Mini_Keystone_3568
Changed lines of the file:
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@@
     (property "Reference" "F5" (id 0) (at 92.71 46.99 90))
     (property "Value" "Fuse" (id 1) (at 92.71 49.53 90))
-    (property "Footprint" "Fuse:Fuse_Blade_Mini_directSolder" (id 2) (at 92.71 55.118 90)
+    (property "Footprint" "Fuse:Fuseholder_Blade_Mini_Keystone_3568" (id 2) (at 92.71 55.118 90)
       (effects (font (size 1.27 1.27)) hide)
     )
@@
     (property "Reference" "F12" (id 0) (at 173.99 116.84 90))
     (property "Value" "Fuse" (id 1) (at 173.99 119.38 90))
-    (property "Footprint" "Fuse:Fuse_Blade_Mini_directSolder" (id 2) (at 173.99 124.968 90)
+    (property "Footprint" "Fuse:Fuseholder_Blade_Mini_Keystone_3568" (id 2) (at 173.99 124.968 90)
       (effects (font (size 1.27 1.27)) hide)
     )
@@
     (property "Reference" "F11" (id 0) (at 173.99 88.9 90))
     (property "Value" "Fuse" (id 1) (at 173.99 91.44 90))
-    (property "Footprint" "Fuse:Fuse_Blade_Mini_directSolder" (id 2) (at 173.99 97.028 90)
+    (property "Footprint" "Fuse:Fuseholder_Blade_Mini_Keystone_3568" (id 2) (at 173.99 97.028 90)
       (effects (font (size 1.27 1.27)) hide)
     )
@@
     (property "Reference" "F7" (id 0) (at 92.71 119.38 90))
     (property "Value" "Fuse" (id 1) (at 92.71 121.92 90))
-    (property "Footprint" "Fuse:Fuse_Blade_Mini_directSolder" (id 2) (at 92.71 127.508 90)
+    (property "Footprint" "Fuse:Fuseholder_Blade_Mini_Keystone_3568" (id 2) (at 92.71 127.508 90)
       (effects (font (size 1.27 1.27)) hide)
     )
@@
     (property "Reference" "F6" (id 0) (at 92.71 67.31 90))
     (property "Value" "Fuse" (id 1) (at 92.71 69.85 90))
-    (property "Footprint" "Fuse:Fuse_Blade_Mini_directSolder" (id 2) (at 92.71 75.438 90)
+    (property "Footprint" "Fuse:Fuseholder_Blade_Mini_Keystone_3568" (id 2) (at 92.71 75.438 90)
       (effects (font (size 1.27 1.27)) hide)
     )
@@
     (property "Reference" "F1" (id 0) (at 85.09 44.45 90))
     (property "Value" "Fuse" (id 1) (at 85.09 46.99 90))
-    (property "Footprint" "Fuse:Fuse_Blade_Mini_directSolder" (id 2) (at 85.09 52.578 90)
+    (property "Footprint" "Fuse:Fuseholder_Blade_Mini_Keystone_3568" (id 2) (at 85.09 52.578 90)
       (effects (font (size 1.27 1.27)) hide)
     )
@@
     (property "Reference" "F9" (id 0) (at 173.99 44.45 90))
     (property "Value" "Fuse" (id 1) (at 173.99 46.99 90))
-    (property "Footprint" "Fuse:Fuse_Blade_Mini_directSolder" (id 2) (at 173.99 52.578 90)
+    (property "Footprint" "Fuse:Fuseholder_Blade_Mini_Keystone_3568" (id 2) (at 173.99 52.578 90)
       (effects (font (size 1.27 1.27)) hide)
     )
@@
     (property "Reference" "F2" (id 0) (at 85.09 64.77 90))
     (property "Value" "Fuse" (id 1) (at 85.09 67.31 90))
-    (property "Footprint" "Fuse:Fuse_Blade_Mini_directSolder" (id 2) (at 85.09 72.898 90)
+    (property "Footprint" "Fuse:Fuseholder_Blade_Mini_Keystone_3568" (id 2) (at 85.09 72.898 90)
       (effects (font (size 1.27 1.27)) hide)
     )
@@
     (property "Reference" "F13" (id 0) (at 181.61 46.99 90))
     (property "Value" "Fuse" (id 1) (at 181.61 49.53 90))
-    (property "Footprint" "Fuse:Fuse_Blade_Mini_directSolder" (id 2) (at 181.61 55.118 90)
+    (property "Footprint" "Fuse:Fuseholder_Blade_Mini_Keystone_3568" (id 2) (at 181.61 55.118 90)
       (effects (font (size 1.27 1.27)) hide)
     )
@@
     (property "Reference" "F16" (id 0) (at 181.61 119.38 90))
     (property "Value" "Fuse" (id 1) (at 181.61 121.92 90))
-    (property "Footprint" "Fuse:Fuse_Blade_Mini_directSolder" (id 2) (at 181.61 127.508 90)
+    (property "Footprint" "Fuse:Fuseholder_Blade_Mini_Keystone_3568" (id 2) (at 181.61 127.508 90)
       (effects (font (size 1.27 1.27)) hide)
     )
@@
     (property "Reference" "F4" (id 0) (at 86.36 88.9 90))
     (property "Value" "Fuse" (id 1) (at 86.36 91.44 90))
-    (property "Footprint" "Fuse:Fuse_Blade_Mini_directSolder" (id 2) (at 86.36 97.028 90)
+    (property "Footprint" "Fuse:Fuseholder_Blade_Mini_Keystone_3568" (id 2) (at 86.36 97.028 90)
       (effects (font (size 1.27 1.27)) hide)
     )
@@
     (property "Reference" "F14" (id 0) (at 181.61 67.31 90))
     (property "Value" "Fuse" (id 1) (at 181.61 69.85 90))
-    (property "Footprint" "Fuse:Fuse_Blade_Mini_directSolder" (id 2) (at 181.61 75.438 90)
+    (property "Footprint" "Fuse:Fuseholder_Blade_Mini_Keystone_3568" (id 2) (at 181.61 75.438 90)
       (effects (font (size 1.27 1.27)) hide)
     )
@@
     (property "Reference" "F10" (id 0) (at 173.99 64.77 90))
     (property "Value" "Fuse" (id 1) (at 173.99 67.31 90))
-    (property "Footprint" "Fuse:Fuse_Blade_Mini_directSolder" (id 2) (at 173.99 72.898 90)
+    (property "Footprint" "Fuse:Fuseholder_Blade_Mini_Keystone_3568" (id 2) (at 173.99 72.898 90)
       (effects (font (size 1.27 1.27)) hide)
     )
@@
     (property "Reference" "F8" (id 0) (at 93.98 91.44 90))
     (property "Value" "Fuse" (id 1) (at 93.98 93.98 90))
-    (property "Footprint" "Fuse:Fuse_Blade_Mini_directSolder" (id 2) (at 93.98 99.568 90)
+    (property "Footprint" "Fuse:Fuseholder_Blade_Mini_Keystone_3568" (id 2) (at 93.98 99.568 90)
       (effects (font (size 1.27 1.27)) hide)
     )
@@
     (property "Reference" "F3" (id 0) (at 85.09 116.84 90))
     (property "Value" "Fuse" (id 1) (at 85.09 119.38 90))
-    (property "Footprint" "Fuse:Fuse_Blade_Mini_directSolder" (id 2) (at 85.09 124.968 90)
+    (property "Footprint" "Fuse:Fuseholder_Blade_Mini_Keystone_3568" (id 2) (at 85.09 124.968 90)
       (effects (font (size 1.27 1.27)) hide)
     )
@@
     (property "Reference" "F15" (id 0) (at 181.61 91.44 90))
     (property "Value" "Fuse" (id 1) (at 181.61 93.98 90))
-    (property "Footprint" "Fuse:Fuse_Blade_Mini_directSolder" (id 2) (at 181.61 99.568 90)
-      (effects (font (size 1.27 1.27)) hide)
-    )
+    (property "Footprint" "Fuse:Fuseholder_Blade_Mini_Keystone_3568" (id 2) (at 181.61 99.568 90)
+      (effects (font (size 1.27 1.27)) hide)
+    )

Commit message: Changed resistors and LEDs to 0805 and updated Production files
Parts:
- D1, D2, D3, D4, D5, D6, D7, D8: footprint LED_SMD:LED_0603_1608Metric -> LED_SMD:LED_0805_2012Metric
- R10, R3, R4, R5, R6, R7, R8, R9: footprint Resistor_SMD:R_0603_1608Metric -> Resistor_SMD:R_0805_2012Metric
Changed lines of the file:
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@@
       (effects (font (size 1.27 1.27)) hide)
     )
-    (property "Footprint" "LED_SMD:LED_0603_1608Metric" (id 2) (at 171.45 102.87 90)
+    (property "Footprint" "LED_SMD:LED_0805_2012Metric" (id 2) (at 171.45 102.87 90)
       (effects (font (size 1.27 1.27)) hide)
     )
@@
     (property "Reference" "R9" (id 0) (at 179.07 105.41 90))
     (property "Value" "10k" (id 1) (at 179.07 100.33 90))
-    (property "Footprint" "Resistor_SMD:R_0603_1608Metric" (id 2) (at 179.324 101.854 90)
+    (property "Footprint" "Resistor_SMD:R_0805_2012Metric" (id 2) (at 179.324 101.854 90)
       (effects (font (size 1.27 1.27)) hide)
     )
@@
     (property "Reference" "R4" (id 0) (at 90.17 81.28 90))
     (property "Value" "10k" (id 1) (at 90.17 76.2 90))
-    (property "Footprint" "Resistor_SMD:R_0603_1608Metric" (id 2) (at 90.424 77.724 90)
+    (property "Footprint" "Resistor_SMD:R_0805_2012Metric" (id 2) (at 90.424 77.724 90)
       (effects (font (size 1.27 1.27)) hide)
     )
@@
       (effects (font (size 1.27 1.27)) hide)
     )
-    (property "Footprint" "LED_SMD:LED_0603_1608Metric" (id 2) (at 82.55 58.42 90)
+    (property "Footprint" "LED_SMD:LED_0805_2012Metric" (id 2) (at 82.55 58.42 90)
       (effects (font (size 1.27 1.27)) hide)
     )
@@
       (effects (font (size 1.27 1.27)) hide)
     )
-    (property "Footprint" "LED_SMD:LED_0603_1608Metric" (id 2) (at 171.45 78.74 90)
+    (property "Footprint" "LED_SMD:LED_0805_2012Metric" (id 2) (at 171.45 78.74 90)
       (effects (font (size 1.27 1.27)) hide)
     )
@@
     (property "Reference" "R10" (id 0) (at 179.07 133.35 90))
     (property "Value" "10k" (id 1) (at 179.07 128.27 90))
-    (property "Footprint" "Resistor_SMD:R_0603_1608Metric" (id 2) (at 179.324 129.794 90)
+    (property "Footprint" "Resistor_SMD:R_0805_2012Metric" (id 2) (at 179.324 129.794 90)
       (effects (font (size 1.27 1.27)) hide)
     )
@@
       (effects (font (size 1.27 1.27)) hide)
     )
-    (property "Footprint" "LED_SMD:LED_0603_1608Metric" (id 2) (at 171.45 130.81 90)
+    (property "Footprint" "LED_SMD:LED_0805_2012Metric" (id 2) (at 171.45 130.81 90)
       (effects (font (size 1.27 1.27)) hide)
     )
@@
     (property "Reference" "R3" (id 0) (at 90.17 60.96 90))
     (property "Value" "10k" (id 1) (at 90.17 55.88 90))
-    (property "Footprint" "Resistor_SMD:R_0603_1608Metric" (id 2) (at 90.424 57.404 90)
+    (property "Footprint" "Resistor_SMD:R_0805_2012Metric" (id 2) (at 90.424 57.404 90)
       (effects (font (size 1.27 1.27)) hide)
     )
@@
       (effects (font (size 1.27 1.27)) hide)
     )
-    (property "Footprint" "LED_SMD:LED_0603_1608Metric" (id 2) (at 82.55 78.74 90)
+    (property "Footprint" "LED_SMD:LED_0805_2012Metric" (id 2) (at 82.55 78.74 90)
       (effects (font (size 1.27 1.27)) hide)
     )
@@
       (effects (font (size 1.27 1.27)) hide)
     )
-    (property "Footprint" "LED_SMD:LED_0603_1608Metric" (id 2) (at 83.82 102.87 90)
+    (property "Footprint" "LED_SMD:LED_0805_2012Metric" (id 2) (at 83.82 102.87 90)
       (effects (font (size 1.27 1.27)) hide)
     )
@@
     (property "Reference" "R5" (id 0) (at 90.17 133.35 90))
     (property "Value" "10k" (id 1) (at 90.17 128.27 90))
-    (property "Footprint" "Resistor_SMD:R_0603_1608Metric" (id 2) (at 90.424 129.794 90)
+    (property "Footprint" "Resistor_SMD:R_0805_2012Metric" (id 2) (at 90.424 129.794 90)
       (effects (font (size 1.27 1.27)) hide)
     )
@@
     (property "Reference" "R8" (id 0) (at 179.07 81.28 90))
     (property "Value" "10k" (id 1) (at 179.07 76.2 90))
-    (property "Footprint" "Resistor_SMD:R_0603_1608Metric" (id 2) (at 179.324 77.724 90)
+    (property "Footprint" "Resistor_SMD:R_0805_2012Metric" (id 2) (at 179.324 77.724 90)
       (effects (font (size 1.27 1.27)) hide)
     )
@@
       (effects (font (size 1.27 1.27)) hide)
     )
-    (property "Footprint" "LED_SMD:LED_0603_1608Metric" (id 2) (at 171.45 58.42 90)
+    (property "Footprint" "LED_SMD:LED_0805_2012Metric" (id 2) (at 171.45 58.42 90)
       (effects (font (size 1.27 1.27)) hide)
     )
@@
       (effects (font (size 1.27 1.27)) hide)
     )
-    (property "Footprint" "LED_SMD:LED_0603_1608Metric" (id 2) (at 82.55 130.81 90)
+    (property "Footprint" "LED_SMD:LED_0805_2012Metric" (id 2) (at 82.55 130.81 90)
       (effects (font (size 1.27 1.27)) hide)
     )
@@
     (property "Reference" "R7" (id 0) (at 179.07 60.96 90))
     (property "Value" "10k" (id 1) (at 179.07 55.88 90))
-    (property "Footprint" "Resistor_SMD:R_0603_1608Metric" (id 2) (at 179.324 57.404 90)
+    (property "Footprint" "Resistor_SMD:R_0805_2012Metric" (id 2) (at 179.324 57.404 90)
       (effects (font (size 1.27 1.27)) hide)
     )
@@
     (property "Reference" "R6" (id 0) (at 91.44 105.41 90))
     (property "Value" "10k" (id 1) (at 91.44 100.33 90))
-    (property "Footprint" "Resistor_SMD:R_0603_1608Metric" (id 2) (at 91.694 101.854 90)
-      (effects (font (size 1.27 1.27)) hide)
-    )
+    (property "Footprint" "Resistor_SMD:R_0805_2012Metric" (id 2) (at 91.694 101.854 90)
+      (effects (font (size 1.27 1.27)) hide)
+    )
