File: PowerBackup/Connectors.kicad_sch (KiCad schematic)
At the start: 8 parts

Commit message: Did some initial board layout
Parts:
- removed J?: Conn_01x02_Female, symbol Connector:Conn_01x02_Female
- removed J? (x2): Conn_01x04_Male, symbol Connector:Conn_01x04_Male
- removed R? (x2): 4k7, symbol Device:R_US
- removed R? (x2): 0, symbol Device:R_US
Other:
- note removed: "Desolder if using I2C LTC4311 board"
