File: PowerBackup/BatteryMonitoring.kicad_sch (KiCad schematic)
At the start: 34 parts, among them J2 Conn_01x07_Male, J3 Conn_01x04_Male, J4 Conn_01x05_Female, J5 Conn_01x04_Male, J6 Conn_01x02_Female, Q1 ZXTP25040DFH, U1 BQ76925RGET

Commit message: Added 5V 9A buck converter
Parts:
- C1, C2, C3, C4, C5, C6, C7, C8, C9: footprint Capacitor_SMD:C_0805_2012Metric -> Capacitor_SMD:C_0603_1608Metric
Connections:
- net at U1.9 (VC0): now also C1.1, R4.2
Changed lines of the file:
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@@
       (effects (font (size 1.27 1.27)) (justify left))
     )
-    (property "Footprint" "Capacitor_SMD:C_0805_2012Metric" (id 2) (at 107.696 103.124 0)
+    (property "Footprint" "Capacitor_SMD:C_0603_1608Metric" (id 2) (at 107.696 103.124 0)
       (effects (font (size 1.27 1.27)) hide)
     )
@@
       (effects (font (size 1.27 1.27)) (justify left))
     )
-    (property "Footprint" "Capacitor_SMD:C_0805_2012Metric" (id 2) (at 92.202 103.124 0)
+    (property "Footprint" "Capacitor_SMD:C_0603_1608Metric" (id 2) (at 92.202 103.124 0)
       (effects (font (size 1.27 1.27)) hide)
     )
@@
       (effects (font (size 1.27 1.27)) (justify left))
     )
-    (property "Footprint" "Capacitor_SMD:C_0805_2012Metric" (id 2) (at 99.822 103.124 0)
+    (property "Footprint" "Capacitor_SMD:C_0603_1608Metric" (id 2) (at 99.822 103.124 0)
       (effects (font (size 1.27 1.27)) hide)
     )
@@
       (effects (font (size 1.27 1.27)) (justify left))
     )
-    (property "Footprint" "Capacitor_SMD:C_0805_2012Metric" (id 2) (at 84.328 103.124 0)
+    (property "Footprint" "Capacitor_SMD:C_0603_1608Metric" (id 2) (at 84.328 103.124 0)
       (effects (font (size 1.27 1.27)) hide)
     )
@@
       (effects (font (size 1.27 1.27)) (justify left))
     )
-    (property "Footprint" "Capacitor_SMD:C_0805_2012Metric" (id 2) (at 162.306 67.056 0)
+    (property "Footprint" "Capacitor_SMD:C_0603_1608Metric" (id 2) (at 162.306 67.056 0)
       (effects (font (size 1.27 1.27)) hide)
     )
@@
       (effects (font (size 1.27 1.27)) (justify left))
     )
-    (property "Footprint" "Capacitor_SMD:C_0805_2012Metric" (id 2) (at 68.834 103.124 0)
+    (property "Footprint" "Capacitor_SMD:C_0603_1608Metric" (id 2) (at 68.834 103.124 0)
       (effects (font (size 1.27 1.27)) hide)
     )
@@
       (effects (font (size 1.27 1.27)) (justify left))
     )
-    (property "Footprint" "Capacitor_SMD:C_0805_2012Metric" (id 2) (at 115.316 103.124 0)
+    (property "Footprint" "Capacitor_SMD:C_0603_1608Metric" (id 2) (at 115.316 103.124 0)
       (effects (font (size 1.27 1.27)) hide)
     )
@@
       (effects (font (size 1.27 1.27)) (justify left))
     )
-    (property "Footprint" "Capacitor_SMD:C_0805_2012Metric" (id 2) (at 76.708 103.124 0)
+    (property "Footprint" "Capacitor_SMD:C_0603_1608Metric" (id 2) (at 76.708 103.124 0)
       (effects (font (size 1.27 1.27)) hide)
     )
@@
       (effects (font (size 1.27 1.27)) (justify left))
     )
-    (property "Footprint" "Capacitor_SMD:C_0805_2012Metric" (id 2) (at 117.856 70.866 0)
-      (effects (font (size 1.27 1.27)) hide)
-    )
+    (property "Footprint" "Capacitor_SMD:C_0603_1608Metric" (id 2) (at 117.856 70.866 0)
+      (effects (font (size 1.27 1.27)) hide)
+    )

Commit message: Looking over desing
Parts:
- J3, J5: footprint (none) -> Connector_JST:JST_SH_BM04B-SRSS-TB_1x04-1MP_P1.00mm_Vertical
Connections:
- net at U1.9 (VC0): now also C1.1, R4.2
Changed lines of the file:
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@@
       (effects (font (size 1.27 1.27)) hide)
     )
-    (property "Footprint" "" (id 2) (at 211.328 74.676 0)
+    (property "Footprint" "Connector_JST:JST_SH_BM04B-SRSS-TB_1x04-1MP_P1.00mm_Vertical" (id 2) (at 211.328 74.676 0)
       (effects (font (size 1.27 1.27)) hide)
     )
@@
       (effects (font (size 1.27 1.27)) hide)
     )
-    (property "Footprint" "" (id 2) (at 237.998 74.676 0)
+    (property "Footprint" "Connector_JST:JST_SH_BM04B-SRSS-TB_1x04-1MP_P1.00mm_Vertical" (id 2) (at 237.998 74.676 0)
       (effects (font (size 1.27 1.27)) hide)
     )

Commit message: Added BOM and production files
Parts:
- added R24: 100, Resistor_SMD:R_0805_2012Metric, symbol Device:R_US
- C1, C2, C3, C4, C5, C6, C7: MFN# (none) -> C1608X6S1H105K080AC
- C8: MFN# (none) -> C0603C104K5RECAUTO
- C9: MFN# (none) -> CL10A475KP8NNNC
- J2, J3, J4, J5, J6, R11, R16, R17: MFN# (none) -> -
- Q1: MFN# (none) -> ZXTP25040DFH; now left out of the parts list
- R1, R2, R3, R4, R5, R6, R7, R8: MFN# (none) -> RMCF0805FT100R
- R10: MFG# CSRL3-0R001F8 -> (none); MFN# (none) -> CSRL3-0R001F8
- R12, R9: footprint Resistor_SMD:R_0805_2012Metric -> Resistor_SMD:R_0603_1608Metric; MFN# (none) -> RNCP0603FTD10K0
- R13, R15: MFN# (none) -> CRGCQ0805J4K7
- R14: value 200 -> 100; MFN# (none) -> RMCF0805FT100R
- TH1: value Thermistor_NTC -> 10k; MFN# (none) -> RNCP0603FTD10K0
- U1: MFN# (none) -> BQ76925RGET
Connections:
- net GNDS is gone; now on net GND: C1.2, C2.2, C3.2, C4.2, C5.2, C6.2, C7.2, C8.2, C9.2, J3.1 (Pin_1), J5.1 (Pin_1), R10.2, R12.2, TH1.2, U1.10 (VSS)
- net SCL: now reaches J3.4 (Pin_3), R13.1, R16.2, U1.19 (SCL)
- net at U1.16 (VTB): now also R24.1; no longer R14.1
- net SDA: now reaches J3.3 (Pin_4), R15.1, R17.2, U1.18 (SDA)
- net at U1.9 (VC0): now also C1.1, R4.2
- new net: R14.1, R24.2
Other:
- note added: "DNL"
- note added: "Replace R11 with 200k if using PNP (Q1)"
- note removed: "Replace with 200k if using PMOS"
- moved on the sheet: C9, Q1

Commit message: Pvin is connected to Vin through a 2.21R resistor
Connections:
- net at U1.9 (VC0): now also C1.1, R4.2
