File: PowerBackup/BatteryMonitoring.kicad_sch (KiCad schematic)
At the start: 35 parts, among them J2 Conn_01x07_Male, J3 Conn_01x04_Male, J4 Conn_01x05_Female, J5 Conn_01x04_Male, J6 Conn_01x02_Female, Q1 ZXTP25040DFH, U1 BQ76925RGET

Commit message: Commiting before order, Regenerated gerbers for both boards
Connections:
- net at U1.9 (VC0): now also C1.1, R4.2
Changed lines of the file:
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@@
   (symbol (lib_id "Device:R_US") (at 225.044 86.36 270) (unit 1)
     (in_bom yes) (on_board yes)
-    (property "Reference" "R17" (id 0) (at 226.314 88.646 90))
-    (property "Value" "0" (id 1) (at 224.028 88.646 90))
+    (property "Reference" "R17" (id 0) (at 230.505 88.265 90))
+    (property "Value" "0" (id 1) (at 221.615 88.265 90))
     (property "Footprint" "Resistor_SMD:R_0805_2012Metric" (id 2) (at 224.79 87.376 90)
       (effects (font (size 1.27 1.27)) hide)
