File: PowerBackup/PowerBackup.kicad_pcb (KiCad board)
At the start: 4 copper layers, 40 x 41 mm, 72 parts, among them J1 Conn_01x02_Female, J10 Conn_01x02_Female, J2 Conn_01x07_Male, J3 Conn_01x04_Male, J4 Conn_01x05_Female, J5 Conn_01x04_Male, J6 Conn_01x02_Female, J7 Conn_01x02_Male, J8 Conn_01x02_Female, J9 Conn_01x02_Female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

Commit message: Commiting before order, Regenerated gerbers for both boards
Routing:
- net GND: vias 89 -> 90
Changed lines of the file:
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@@
     (fp_line (start -0.625 -2.35) (end 0 -1.35) (layer "F.Fab") (width 0.1))
     (fp_line (start 4.95 -2.35) (end -2.45 -2.35) (layer "F.Fab") (width 0.1))
-    (pad "1" thru_hole roundrect (at 0 0 90) (size 1.7 2) (drill 1) (layers *.Cu *.Mask) (roundrect_rratio 0.1470588235)
+    (pad "1" thru_hole roundrect (at 0 0 90) (size 1.7 2) (drill 1.5) (layers *.Cu *.Mask) (roundrect_rratio 0.1470588235)
       (net 38 "+5V") (pinfunction "Pin_1") (pintype "passive"))
-    (pad "2" thru_hole oval (at 2.5 0 90) (size 1.7 2) (drill 1) (layers *.Cu *.Mask)
+    (pad "2" thru_hole oval (at 2.5 0 90) (size 1.7 2) (drill 1.5) (layers *.Cu *.Mask)
       (net 2 "GND") (pinfunction "Pin_2") (pintype "passive"))
     (model "${KICAD6_3DMODEL_DIR}/Connector_JST.3dshapes/JST_XH_B2B-XH-A_1x02_P2.50mm_Vertical.wrl"
@@
     (fp_line (start 0 -1.35) (end 0.625 -2.35) (layer "F.Fab") (width 0.1))
     (fp_line (start -2.45 -2.35) (end -2.45 3.4) (layer "F.Fab") (width 0.1))
-    (pad "1" thru_hole roundrect (at 0 0 180) (size 1.7 2) (drill 1) (layers *.Cu *.Mask) (roundrect_rratio 0.1470588235)
+    (pad "1" thru_hole roundrect (at 0 0 180) (size 1.7 2) (drill 1.5) (layers *.Cu *.Mask) (roundrect_rratio 0.1470588235)
       (net 38 "+5V") (pinfunction "Pin_1") (pintype "passive"))
-    (pad "2" thru_hole oval (at 2.5 0 180) (size 1.7 2) (drill 1) (layers *.Cu *.Mask)
+    (pad "2" thru_hole oval (at 2.5 0 180) (size 1.7 2) (drill 1.5) (layers *.Cu *.Mask)
       (net 2 "GND") (pinfunction "Pin_2") (pintype "passive"))
     (model "${KICAD6_3DMODEL_DIR}/Connector_JST.3dshapes/JST_XH_B2B-XH-A_1x02_P2.50mm_Vertical.wrl"
@@
     (fp_line (start -2.45 -2.35) (end -2.45 3.4) (layer "F.Fab") (width 0.1))
     (fp_line (start 4.95 -2.35) (end -2.45 -2.35) (layer "F.Fab") (width 0.1))
-    (pad "1" thru_hole roundrect (at 0 0) (size 1.7 2) (drill 1) (layers *.Cu *.Mask) (roundrect_rratio 0.1470588235)
+    (pad "1" thru_hole roundrect (at 0 0) (size 1.7 2) (drill 1.5) (layers *.Cu *.Mask) (roundrect_rratio 0.1470588235)
       (net 34 "/Backup/VBAT") (pinfunction "Pin_1") (pintype "passive"))
-    (pad "2" thru_hole oval (at 2.5 0) (size 1.7 2) (drill 1) (layers *.Cu *.Mask)
+    (pad "2" thru_hole oval (at 2.5 0) (size 1.7 2) (drill 1.5) (layers *.Cu *.Mask)
       (net 2 "GND") (pinfunction "Pin_2") (pintype "passive"))
     (model "${KICAD6_3DMODEL_DIR}/Connector_JST.3dshapes/JST_XH_B2B-XH-A_1x02_P2.50mm_Vertical.wrl"
@@
     (fp_line (start -0.625 -2.35) (end 0 -1.35) (layer "F.Fab") (width 0.1))
     (fp_line (start 0 -1.35) (end 0.625 -2.35) (layer "F.Fab") (width 0.1))
-    (pad "1" thru_hole roundrect (at 0 0 180) (size 1.7 2) (drill 1) (layers *.Cu *.Mask) (roundrect_rratio 0.1470588235)
+    (pad "1" thru_hole roundrect (at 0 0 180) (size 1.7 2) (drill 1.5) (layers *.Cu *.Mask) (roundrect_rratio 0.1470588235)
       (net 38 "+5V") (pinfunction "Pin_1") (pintype "passive"))
-    (pad "2" thru_hole oval (at 2.5 0 180) (size 1.7 2) (drill 1) (layers *.Cu *.Mask)
+    (pad "2" thru_hole oval (at 2.5 0 180) (size 1.7 2) (drill 1.5) (layers *.Cu *.Mask)
       (net 2 "GND") (pinfunction "Pin_2") (pintype "passive"))
     (model "${KICAD6_3DMODEL_DIR}/Connector_JST.3dshapes/JST_XH_B2B-XH-A_1x02_P2.50mm_Vertical.wrl"
@@
     (fp_line (start 0 1.35) (end 0.625 2.35) (layer "B.Fab") (width 0.1))
     (fp_line (start -2.45 2.35) (end -2.45 -3.4) (layer "B.Fab") (width 0.1))
-    (pad "1" thru_hole roundrect (at 0 0 180) (size 1.7 2) (drill 1) (layers *.Cu *.Mask) (roundrect_rratio 0.1470588235)
+    (pad "1" thru_hole roundrect (at 0 0 180) (size 1.7 2) (drill 1.5) (layers *.Cu *.Mask) (roundrect_rratio 0.1470588235)
       (net 11 "+9V") (pinfunction "Pin_1") (pintype "passive"))
-    (pad "2" thru_hole oval (at 2.5 0 180) (size 1.7 2) (drill 1) (layers *.Cu *.Mask)
+    (pad "2" thru_hole oval (at 2.5 0 180) (size 1.7 2) (drill 1.5) (layers *.Cu *.Mask)
       (net 2 "GND") (pinfunction "Pin_2") (pintype "passive"))
     (model "${KICAD6_3DMODEL_DIR}/Connector_JST.3dshapes/JST_XH_B2B-XH-A_1x02_P2.50mm_Vertical.wrl"
@@
   (via (at 149.25 94.85) (size 0.8) (drill 0.4) (layers "F.Cu" "B.Cu") (free) (net 2))
   (via (at 112.6 88.6) (size 0.8) (drill 0.4) (layers "F.Cu" "B.Cu") (net 2))
+  (via (at 134.8 111.3) (size 0.8) (drill 0.4) (layers "F.Cu" "B.Cu") (free) (net 2))
   (via (at 128.6 95) (size 0.8) (drill 0.4) (layers "F.Cu" "B.Cu") (free) (net 2))
   (via (at 149.352 96.266) (size 0.8) (drill 0.4) (layers "F.Cu" "B.Cu") (free) (net 2))
